File: hardware/KiCad/zx-rgbi-to-vga-hdmi_gotek-osd_keyboard.kicad_sch (KiCad schematic)
At the start: 30 parts, among them J1 HDMI_A, J2 VGA, J3 ZX KEYBOARD, J4 PS/2 KEYBOARD, J5 GOTEK I2C, J6 CAP_0, U1 Pico, U2 CH446Q, U3 74LVC245A

Commit message: Connect +5V to CH446Q VDD.
Connections:
- net +5V: now also C3.1, U2.38 (VDD)
Changed lines of the file:
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@@
+		)
+	)
+	(label "+5V"
+		(at 242.57 116.84 0)
+		(fields_autoplaced yes)
+		(effects
+			(font
+				(size 1.27 1.27)
+			)
+			(justify left bottom)
 		)
 	)
