File: hardware/KiCad/zx-rgbi-to-vga-hdmi_gotek-osd_keyboard.kicad_sch (KiCad schematic)
At the start: 30 parts, among them J1 HDMI_A, J2 VGA, J3 ZX KEYBOARD, J4 PS/2 KEYBOARD, J5 GOTEK I2C, J6 CAP_0, U1 Pico, U2 CH446Q, U3 74LVC245A

Commit message: CH446Q output Z80 control signals PAUSE, MAGIC, RESET have common input connected to GND.
Connections:
- net GND: now also U2.5 (X8)
- no-connect marks 31 -> 30
Changed lines of the file:
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@@
 	)
 	(no_connect
-		(at 250.19 33.02)
-	)
-	(no_connect
 		(at 250.19 22.86)
 	)
@@
 					(unit 1)
 				)
+			)
+		)
+	)
+	(symbol
+		(lib_id "power:GND")
+		(at 250.19 33.02 270)
+		(unit 1)
+		(exclude_from_sim no)
+		(in_bom yes)
+		(on_board yes)
+		(dnp no)
+		(fields_autoplaced yes)
+		(property "Reference" "#PWR015"
+			(at 243.84 33.02 0)
+			(effects
+				(font
+					(size 1.27 1.27)
+				)
+				(hide yes)
+			)
+		)
+		(property "Value" "GND"
+			(at 246.38 33.0199 90)
+			(effects
+				(font
+					(size 1.27 1.27)
+				)
+				(justify right)
+			)
+		)
+		(property "Footprint" ""
+			(at 250.19 33.02 0)
+			(effects
+				(font
+					(size 1.27 1.27)
+				)
+				(hide yes)
+			)
+		)
+		(property "Datasheet" ""
+			(at 250.19 33.02 0)
+			(effects
+				(font
+					(size 1.27 1.27)
+				)
+				(hide yes)
+			)
+		)
+		(property "Description" "Power symbol creates a global label with name \"GND\" , ground"
+			(at 250.19 33.02 0)
+			(effects
+				(font
+					(size 1.27 1.27)
+				)
+				(hide yes)
+			)
+		)
+		(pin "1"
+		)
+		(instances
+			(project "zx-rgbi-to-vga-hdmi_gotek-osd_keyboard"
+				(path "/ea33e844-7ede-417a-b45b-9c2bb2acafa2"
+					(reference "#PWR015")
+					(unit 1)
+				)

Commit message: Change schematic for BOARD_CODE_36LJU22 (capture pins starts from GP0, HDMI/VGA data lines starts from GP8).
Connections:
- net GP0: now also U3.17 (B1)
- net GP1: now also U3.16 (B2)
- net GP10: now also R3.2; no longer U3.12 (B6)
- net GP11: now also R4.2; no longer U3.11 (B7)
- net GP12: now also R5.2; no longer R1.2
- net GP13: now also R6.2; no longer R2.2
- net GP14: now also R7.2; no longer R3.2
- net GP15: now also R8.2; no longer R4.2
- net GP16: no longer R5.2
- net GP17: no longer R6.2
- net GP18: no longer R7.2
- net GP19: no longer R8.2
- net GP2: now also U3.15 (B3)
- net GP3: now also U3.14 (B4)
- net GP4: now also U3.13 (B5)
- net GP5: now also U3.12 (B6); no longer U3.17 (B1)
- net GP6: now also U3.11 (B7); no longer U3.16 (B2)
- net GP7: no longer U3.15 (B3)
- net GP8: now also R1.2; no longer U3.14 (B4)
- net GP9: now also R2.2; no longer U3.13 (B5)
Changed lines of the file:
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@@
 		)
 	)
-	(label "GP8"
+	(label "GP3"
 		(at 180.34 60.96 0)
 		(fields_autoplaced yes)
@@
 		)
 	)
-	(label "GP17"
+	(label "GP13"
 		(at 95.25 72.39 0)
 		(fields_autoplaced yes)
@@
 		)
 	)
-	(label "GP6"
+	(label "GP1"
 		(at 180.34 55.88 0)
 		(fields_autoplaced yes)
@@
 		)
 	)
-	(label "GP11"
+	(label "GP6"
 		(at 180.34 68.58 0)
 		(fields_autoplaced yes)
@@
 		)
 	)
-	(label "GP5"
+	(label "GP0"
 		(at 180.34 53.34 0)
 		(fields_autoplaced yes)
@@
 		)
 	)
-	(label "GP7"
+	(label "GP2"
 		(at 180.34 58.42 0)
 		(fields_autoplaced yes)
@@
 		)
 	)
-	(label "GP9"
+	(label "GP4"
 		(at 180.34 63.5 0)
 		(fields_autoplaced yes)
@@
 		)
 	)
-	(label "GP19"
+	(label "GP15"
 		(at 95.25 77.47 0)
 		(fields_autoplaced yes)
@@
 		)
 	)
-	(label "GP15"
+	(label "GP11"
 		(at 95.25 67.31 0)
 		(fields_autoplaced yes)
@@
 		)
 	)
-	(label "GP14"
+	(label "GP10"
 		(at 95.25 64.77 0)
 		(fields_autoplaced yes)
@@
 		)
 	)
-	(label "GP12"
+	(label "GP8"
 		(at 95.25 59.69 0)
 		(fields_autoplaced yes)
@@
 		)
 	)
-	(label "GP18"
+	(label "GP14"
 		(at 95.25 74.93 0)
 		(fields_autoplaced yes)
@@
 		)
 	)
-	(label "GP13"
+	(label "GP9"
 		(at 95.25 62.23 0)
 		(fields_autoplaced yes)
@@
 		)
 	)
-	(label "GP10"
+	(label "GP5"
 		(at 180.34 66.04 0)
 		(fields_autoplaced yes)
@@
 		)
 	)
-	(label "GP16"
+	(label "GP12"
 		(at 95.25 69.85 0)
 		(fields_autoplaced yes)
